File: pico_vga_sd_aud/pico_vga_sd_aud.kicad_pcb (KiCad board)
At the start: 4 copper layers, 85 x 56 mm, 71 parts, among them J1 AudioJack3, J2 AudioJack3, J3 Micro_SD_Card, J4 L77HDE15SD1CH4F, J5 USB_B_Micro, J6 Conn_01x02, J7 Conn_02x03_Odd_Even, SW1 SW_Push, SW2 SW_Push, SW3 SW_Push, SW4 SW_Push, U1 TLV70033_SOT23-5, U2 Pico, U3 NC7WZ16P6X, U4 PCM5101A

Commit message: picow: Upgrade project to Verison 7.0.9
Fix missing symbols. Remove old project files.
Other:
- net class Default removed

Commit message: pico: Update footprint to new one with a keepout
Update symbol to new one
Parts:
- U2: footprint RPi_Pico:RPi_Pico_SMD_TH -> RaspberryPi_Pico_SMD:RPi_Pico_SMD
Connections:
- net +3V3 renamed +3.3V
- J3 pad 10: Net-(J3-Pad10) -> unconnected-(J3-DET_A-Pad10)
- J3 pad 9: Net-(J3-Pad9) -> unconnected-(J3-DET_B-Pad9)
- J4 pad 11: Net-(J4-Pad11) -> unconnected-(J4-Pad11)
- J4 pad 12: Net-(J4-Pad12) -> unconnected-(J4-Pad12)
- J4 pad 15: Net-(J4-Pad15) -> unconnected-(J4-Pad15)
- J4 pad 4: Net-(J4-Pad4) -> unconnected-(J4-Pad4)
- J4 pad 9: Net-(J4-Pad9) -> unconnected-(J4-Pad9)
- J5 pad 2: Net-(J5-Pad2) -> unconnected-(J5-D--Pad2)
- J5 pad 3: Net-(J5-Pad3) -> unconnected-(J5-D+-Pad3)
- J5 pad 4: Net-(J5-Pad4) -> unconnected-(J5-ID-Pad4)
- U1 pad 4: Net-(U1-Pad4) -> unconnected-(U1-NC-Pad4)
- U2 pad 35: Net-(U2-Pad35) -> unconnected-(U2-ADC_VREF-Pad35)
- U2 pad 37: Net-(U2-Pad37) -> unconnected-(U2-3V3_EN-Pad37)
