File: picow_vga_sd_aud/picow_vga_sd_aud.kicad_pcb (KiCad board)
At the start: 4 copper layers, 74 x 52 mm, 52 parts, among them J2 AudioJack3, J3 Micro_SD_Card, J4 L77HDE15SD1CH4F, J7 Conn_02x03_Odd_Even, SW1 SW_Push, SW2 SW_Push, SW3 SW_Push, SW4 SW_Push, U1 TLV70033_SOT23-5, U2 PicoW, U3 NC7WZ16P6X

Commit message: picow: Update new footprint (with keepout) and symbol
Parts:
- U2: footprint RaspberryPI PicoW:RPi_PicoW_SMD_TH -> RaspberryPi_Pico_SMD:RPi_PicoW_SMD

Commit message: picow: Get ERC to pass
Connections:
- net +3V3 renamed +3.3V
