File: picow_vga_sd_aud/picow_vga_sd_aud.kicad_sch (KiCad schematic)
At the start: 52 parts, among them J2 AudioJack3, J3 Micro_SD_Card, J4 L77HDE15SD1CH4F, J7 Conn_02x03_Odd_Even, SW1 SW_Push, SW2 SW_Push, SW3 SW_Push, SW4 SW_Push, U1 TLV70033_SOT23-5, U2 PicoW, U3 NC7WZ16P6X

Commit message: picow: Update new footprint (with keepout) and symbol
Parts:
- U2: footprint RaspberryPI PicoW:RPi_PicoW_SMD_TH -> RaspberryPi_Pico_SMD:RPi_PicoW_SMD; symbol RPi_Pico:PicoW -> MCU_RaspberryPi_Pico:PicoW
Changed lines of the file:
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@@
     (effects (font (size 1.27 1.27)) (justify right bottom))
   )
-  (symbol (lib_id "RPi_Pico:PicoW") (at 73.66 114.3 0) (unit 1)
+  (symbol (lib_id "MCU_RaspberryPi_Pico:PicoW") (at 73.66 114.3 0) (unit 1)
     (in_bom yes) (on_board yes) (dnp no)
     (property "Reference" "U2" (at 73.66 85.09 0)
@@
       (effects (font (size 1.27 1.27)))
     )
-    (property "Footprint" "RaspberryPI PicoW:RPi_PicoW_SMD_TH" (at 73.66 114.3 90)
+    (property "Footprint" "RaspberryPi_Pico_SMD:RPi_PicoW_SMD" (at 73.66 114.3 90)
       (effects (font (size 1.27 1.27)) hide)
     )

Commit message: picow: Get ERC to pass
Parts:
- J3: symbol Connector:Micro_SD_Card_Det -> Connector:Micro_SD_Card_Det2
- J4: symbol Connector:DB15_Female_HighDensity_MountingHoles -> Connector:DE15_Receptacle_HighDensity_MountingHoles
Connections:
- net +3V3 renamed +3.3V
- no-connect marks 9 -> 10
Changed lines of the file:
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@@
   (junction (at 355.6 90.17) (diameter 0) (color 0 0 0 0)
   )
+  (junction (at 168.91 39.37) (diameter 0) (color 0 0 0 0)
+  )
   (junction (at 355.6 100.33) (diameter 0) (color 0 0 0 0)
   )
@@
   (no_connect (at 373.38 90.17))
   (no_connect (at 336.55 224.79))
+  (no_connect (at 107.95 113.03))
   (no_connect (at 373.38 69.85))
   (wire (pts (xy 132.08 115.57) (xy 134.62 115.57))
@@
     (stroke (width 0) (type default))
   )
+  (wire (pts (xy 168.91 39.37) (xy 160.02 39.37))
+    (stroke (width 0) (type default))
+  )
   (wire (pts (xy 91.44 115.57) (xy 121.92 115.57))
     (stroke (width 0) (type default))
@@
     (stroke (width 0) (type default))
   )
+  (wire (pts (xy 38.1 200.66) (xy 38.1 205.74))
+    (stroke (width 0) (type default))
+  )
   (wire (pts (xy 39.37 97.79) (xy 55.88 97.79))
     (stroke (width 0) (type default))
@@
     (stroke (width 0) (type default))
   )
+  (wire (pts (xy 25.4 200.66) (xy 25.4 205.74))
+    (stroke (width 0) (type default))
+  )
   (wire (pts (xy 358.14 77.47) (xy 355.6 77.47))
     (stroke (width 0) (type default))
@@
     (stroke (width 0) (type default))
   )
+  (wire (pts (xy 160.02 39.37) (xy 160.02 49.53))
+    (stroke (width 0) (type default))
+  )
   (wire (pts (xy 358.14 74.93) (xy 347.98 74.93))
     (stroke (width 0) (type default))
@@
     )
   )
-  (symbol (lib_id "Connector:Micro_SD_Card_Det") (at 359.41 214.63 0) (unit 1)
+  (symbol (lib_id "Connector:Micro_SD_Card_Det2") (at 359.41 214.63 0) (unit 1)
     (in_bom yes) (on_board yes) (dnp no)
     (property "Reference" "J3" (at 341.63 233.68 0)
@@
       (effects (font (size 1.27 1.27)))
     )
-    (property "Footprint" "Connector_Card:microSD_HC_Molex_104031-0811" (at 388.62 207.01 0)
+    (property "Footprint" "Connector_Card:microSD_HC_Molex_104031-0811" (at 411.48 196.85 0)
       (effects (font (size 1.27 1.27)) hide)
     )
-    (property "Datasheet" "http://katalog.we-online.de/em/datasheet/693072010801.pdf" (at 359.41 214.63 0)
+    (property "Datasheet" "https://www.hirose.com/en/product/document?clcode=&productname=&series=DM3&documenttype=Catalog&lang=en&documentid=D49662_en" (at 361.95 212.09 0)
       (effects (font (size 1.27 1.27)) hide)
     )
@@
     )
   )
-  (symbol (lib_id "Connector:DB15_Female_HighDensity_MountingHoles") (at 365.76 80.01 0) (unit 1)
+  (symbol (lib_id "Connector:DE15_Receptacle_HighDensity_MountingHoles") (at 365.76 80.01 0) (unit 1)
     (in_bom yes) (on_board yes) (dnp no)
     (property "Reference" "J4" (at 365.76 57.9882 0)
@@
       (effects (font (size 1.27 1.27)) hide)
     )
-    (pin "0")
     (pin "1")
     (pin "10")
@@
     (pin "8")
     (pin "9")
+    (pin "0")
     (instances
       (project "picow_vga_sd_aud"
@@
       (effects (font (size 1.27 1.27)) hide)
     )
-    (property "Value" "GND" (at 168.783 53.9242 0)
+    (property "Value" "GND" (at 168.91 54.61 0)
       (effects (font (size 1.27 1.27)))
     )
@@
         )
       )
+    )
+  )
+  (symbol (lib_id "power:PWR_FLAG") (at 38.1 205.74 180) (unit 1)
+    (in_bom yes) (on_board yes) (dnp no) (fields_autoplaced)
+    (property "Reference" "#FLG03" (at 38.1 207.645 0)
+      (effects (font (size 1.27 1.27)) hide)
+    )
+    (property "Value" "PWR_FLAG" (at 38.1 210.82 0)
+      (effects (font (size 1.27 1.27)))
+    )
+    (property "Footprint" "" (at 38.1 205.74 0)
+      (effects (font (size 1.27 1.27)) hide)
+    )
+    (property "Datasheet" "~" (at 38.1 205.74 0)
+      (effects (font (size 1.27 1.27)) hide)
+    )
+    (pin "1")
+    (instances
+      (project "picow_vga_sd_aud"
+        (path "/7e7c068a-a341-4358-ab45-53bb7a793d6f"
+          (reference "#FLG03") (unit 1)
+        )
+      )
+    )
+  )
+  (symbol (lib_id "power:VBUS") (at 38.1 200.66 0) (unit 1)
+    (in_bom yes) (on_board yes) (dnp no)
+    (property "Reference" "#PWR03" (at 38.1 204.47 0)
+      (effects (font (size 1.27 1.27)) hide)
+    )
+    (property "Value" "VBUS" (at 38.1 195.58 0)
+      (effects (font (size 1.27 1.27)))
+    )
+    (property "Footprint" "" (at 38.1 200.66 0)
+      (effects (font (size 1.27 1.27)) hide)
+    )
+    (property "Datasheet" "" (at 38.1 200.66 0)
+      (effects (font (size 1.27 1.27)) hide)
+    )
+    (pin "1")
+    (instances
+      (project "picow_vga_sd_aud"
+        (path "/7e7c068a-a341-4358-ab45-53bb7a793d6f"
+          (reference "#PWR03") (unit 1)
+        )
+      )
+    )
+  )
+  (symbol (lib_id "power:GND") (at 25.4 205.74 0) (mirror y) (unit 1)
+    (in_bom yes) (on_board yes) (dnp no)
+    (property "Reference" "#PWR01" (at 25.4 212.09 0)
+      (effects (font (size 1.27 1.27)) hide)
+    )
+    (property "Value" "GND" (at 25.4 210.82 0)
+      (effects (font (size 1.27 1.27)))
+    )
+    (property "Footprint" "" (at 25.4 205.74 0)
+      (effects (font (size 1.27 1.27)) hide)
+    )
+    (property "Datasheet" "" (at 25.4 205.74 0)
+      (effects (font (size 1.27 1.27)) hide)
+    )
+    (pin "1")
+    (instances
+      (project "picow_vga_sd_aud"
+        (path "/7e7c068a-a341-4358-ab45-53bb7a793d6f"
+          (reference "#PWR01") (unit 1)
+        )
+      )
+    )
+  )
+  (symbol (lib_id "power:PWR_FLAG") (at 160.02 49.53 180) (unit 1)
+    (in_bom yes) (on_board yes) (dnp no)
+    (property "Reference" "#FLG04" (at 160.02 51.435 0)
+      (effects (font (size 1.27 1.27)) hide)
+    )
+    (property "Value" "PWR_FLAG" (at 160.02 54.61 0)
+      (effects (font (size 1.27 1.27)))
+    )
+    (property "Footprint" "" (at 160.02 49.53 0)
+      (effects (font (size 1.27 1.27)) hide)
+    )
+    (property "Datasheet" "~" (at 160.02 49.53 0)
+      (effects (font (size 1.27 1.27)) hide)
+    )
+    (pin "1")
+    (instances
+      (project "picow_vga_sd_aud"
+        (path "/7e7c068a-a341-4358-ab45-53bb7a793d6f"
+          (reference "#FLG04") (unit 1)
+        )
+      )
+    )
+  )
+  (symbol (lib_id "power:PWR_FLAG") (at 25.4 200.66 0) (unit 1)
+    (in_bom yes) (on_board yes) (dnp no) (fields_autoplaced)
+    (property "Reference" "#FLG01" (at 25.4 198.755 0)
+      (effects (font (size 1.27 1.27)) hide)
+    )
+    (property "Value" "PWR_FLAG" (at 25.4 195.58 0)
+      (effects (font (size 1.27 1.27)))
+    )
+    (property "Footprint" "" (at 25.4 200.66 0)
+      (effects (font (size 1.27 1.27)) hide)
+    )
+    (property "Datasheet" "~" (at 25.4 200.66 0)
+      (effects (font (size 1.27 1.27)) hide)
+    )
+    (pin "1")
+    (instances
+      (project "picow_vga_sd_aud"
+        (path "/7e7c068a-a341-4358-ab45-53bb7a793d6f"
+          (reference "#FLG01") (unit 1)
+        )
+      )
